File: LaserOps_PCB.kicad_pcb (KiCad board)
At the start: 2 copper layers, 0 parts

Commit message: pcb layout designing
Parts:
- added BT2: Li-ion Batterypack (6V-8.4V), Connector_PinHeader_2.54mm:PinHeader_1x02_P2.54mm_Vertical, F.Cu at (147.0, 108.0)
- added C1: 10uF, PCM_JLCPCB:C_CASE-A-3216-18(mm), F.Cu at (196.0, 98.5)
- added C10: 100nF, PCM_JLCPCB:C_0805, F.Cu at (163.1, 96.1)
- added C11: 100nF, PCM_JLCPCB:C_0805, F.Cu at (171.0, 94.7)
- added C12: 22uF, PCM_JLCPCB:C_0805, F.Cu at (171.6, 89.1)
- added C13: 10uF, PCM_JLCPCB:C_0805, F.Cu at (168.9, 94.7)
- added C14: 22uF, PCM_JLCPCB:C_0805, F.Cu at (198.0, 123.0)
- added C15: 22uF, PCM_JLCPCB:C_0805, F.Cu at (171.0, 107.1)
- added C16: 22uF, PCM_JLCPCB:C_0805, F.Cu at (199.8, 118.8)
- added C17: 10uF, PCM_JLCPCB:C_0805, F.Cu at (164.0, 116.4)
- added C18: 22uF, PCM_JLCPCB:C_1206, F.Cu at (105.3, 31.6)
- added C19: 10uF, PCM_JLCPCB:C_1206, F.Cu at (105.3, 35.0)
- added C2: 100nF, PCM_JLCPCB:C_0805, F.Cu at (177.3, 92.3)
- added C20: 100µF, Capacitor_THT:CP_Radial_D5.0mm_P2.50mm, F.Cu at (110.8, 57.4)
- added C21: 220µF, Capacitor_THT:CP_Radial_D6.3mm_P2.50mm, F.Cu at (119.0, 58.6)
- added C22: 100nF, PCM_JLCPCB:C_1206, F.Cu at (105.3, 38.3)
- added C23: 100nF, PCM_JLCPCB:C_1206, F.Cu at (105.3, 41.7)
- added C24: 10uF, PCM_JLCPCB:C_1206, F.Cu at (105.3, 45.0)
- added C25: 22uF, PCM_JLCPCB:C_1206, F.Cu at (105.3, 48.4)
- added C26: 100uF, PCM_JLCPCB:C_1206, F.Cu at (105.3, 51.7)
- added C27: 22pF, PCM_JLCPCB:C_0805, F.Cu at (159.5, 101.0)
- added C28: 100nF, PCM_JLCPCB:C_0805, F.Cu at (164.0, 118.5)
- added C29: 10uF, PCM_JLCPCB:C_0805, F.Cu at (163.1, 98.2)
- added C3: 100nF, PCM_JLCPCB:C_0805, F.Cu at (195.9, 123.0)
- added C30: 10uF, PCM_JLCPCB:C_0805, F.Cu at (168.1, 99.3)
- added C31: 100nF, PCM_JLCPCB:C_0805, F.Cu at (166.0, 99.3)
- added C32: 10uF, PCM_JLCPCB:C_0805, F.Cu at (117.2, 37.0)
- added C33: 100nF, PCM_JLCPCB:C_0805, F.Cu at (117.2, 40.0)
- added C4: 47pF, PCM_JLCPCB:C_0805, F.Cu at (184.1, 95.0)
- added C5: 10uF, PCM_JLCPCB:C_CASE-A-3216-18(mm), F.Cu at (196.0, 100.7)
- added C6: 1uF, PCM_JLCPCB:C_0805, F.Cu at (195.6, 119.8)
- added C7: 22uF, PCM_JLCPCB:C_0805, F.Cu at (171.6, 91.2)
- added C8: 1uF, PCM_JLCPCB:C_0805, F.Cu at (168.9, 107.2)
- added C9: 10uF, PCM_JLCPCB:C_0805, F.Cu at (195.0, 103.0)
- added Camera_Interface1: Conn_02x08_Counter_Clockwise, Connector_JST:JST_PH_B16B-PH-SM4-TB_1x16-1MP_P2.00mm_Vertical, B.Cu at (217.3, 81.0)
- added D1: 1N4002W, PCM_JLCPCB:D_SOD-123FL, F.Cu at (120.1, 30.7)
- added D2: 1N4002W, PCM_JLCPCB:D_SOD-123FL, F.Cu at (120.1, 34.0)
- added J2: Conn_01x02_Socket, Connector_PinHeader_2.54mm:PinHeader_1x02_P2.54mm_Vertical, F.Cu at (162.1, 88.9)
- added J3: Dome, Connector_JST:JST_PH_S6B-PH-SM4-TB_1x06-1MP_P2.00mm_Horizontal, F.Cu at (105.8, 137.6)
- added J4: USB_C_Receptacle_USB2.0_14P, Connector_USB:USB_C_Receptacle_GCT_USB4085, B.Cu at (194.5, 106.7)
- added J5: Motor1, Connector_JST:JST_PH_S2B-PH-SM4-TB_1x02-1MP_P2.00mm_Horizontal, F.Cu at (116.1, 106.5)
- added J6: Motor2, Connector_JST:JST_PH_S2B-PH-SM4-TB_1x02-1MP_P2.00mm_Horizontal, F.Cu at (123.3, 119.7)
- added J7: Speaker, Connector_JST:JST_PH_S2B-PH-SM4-TB_1x02-1MP_P2.00mm_Horizontal, B.Cu at (158.9, 110.7)
- added J8: Conn_01x07, Connector_JST:JST_PH_S7B-PH-SM4-TB_1x07-1MP_P2.00mm_Horizontal, F.Cu at (86.0, 123.0)
- added J9: IR-LED, Connector_PinHeader_2.54mm:PinHeader_1x02_P2.54mm_Vertical, F.Cu at (162.5, 93.2)
- added JP1: Indoor/Outdoor, Jumper:SolderJumper-2_P1.3mm_Open_RoundedPad1.0x1.5mm, F.Cu at (123.1, 36.9)
- added JP5: Jumper, Jumper:SolderJumper-3_P1.3mm_Bridged12_RoundedPad1.0x1.5mm_NumberLabels, F.Cu at (121.7, 52.8)
- added JP6: Jumper, Jumper:SolderJumper-3_P1.3mm_Bridged12_RoundedPad1.0x1.5mm_NumberLabels, F.Cu at (113.4, 30.9)
- added JP7: Jumper, Jumper:SolderJumper-3_P1.3mm_Bridged12_RoundedPad1.0x1.5mm_NumberLabels, F.Cu at (113.4, 34.4)
- added JP8: Jumper, Jumper:SolderJumper-3_P1.3mm_Bridged12_RoundedPad1.0x1.5mm_NumberLabels, B.Cu at (171.8, 98.8)
- added L1: 6.8µH, Inductor_SMD:L_Coilcraft_LPS5030, B.Cu at (169.2, 93.0)
- added Q1: IRLML6344TRPBF, IRLML6344TRPBF:TRANS_IRLML6344TRPBF, B.Cu at (159.4, 97.9)
- added Q2: HL2305, PCM_JLCPCB:Q_SOT-23, F.Cu at (184.4, 98.7)
- added Q8: S9014, PCM_JLCPCB:Q_SOT-23, F.Cu at (113.0, 42.2)
- added Q9: S9014, PCM_JLCPCB:Q_SOT-23, F.Cu at (113.0, 46.8)
- added R1: 5.1kΩ, PCM_JLCPCB:R_0805, F.Cu at (121.7, 41.4)
- added R10: 1Ω 2W, Resistor_SMD:R_2512_6332Metric_Pad1.40x3.35mm_HandSolder, F.Cu at (188.5, 91.5)
- added R11: 5.1kΩ, PCM_JLCPCB:R_0805, F.Cu at (121.7, 44.4)
- added R12: 10kΩ, PCM_JLCPCB:R_0805, F.Cu at (166.8, 107.2)
- added R15: 634k, Resistor_SMD:R_0805_2012Metric_Pad1.20x1.40mm_HandSolder, F.Cu at (166.9, 117.6)
- added R16: 100kΩ, PCM_JLCPCB:R_0805, F.Cu at (175.6, 100.1)
- added R17: 22kΩ, PCM_JLCPCB:R_0805, F.Cu at (180.0, 95.0)
- added R18: 10kΩ, PCM_JLCPCB:R_0805, F.Cu at (195.6, 117.8)
- added R19: 100kΩ, PCM_JLCPCB:R_0805, F.Cu at (184.2, 101.4)
- added R2: 300kΩ, PCM_JLCPCB:R_0805, F.Cu at (180.7, 100.1)
- added R20: 100Ω, PCM_JLCPCB:R_0805, F.Cu at (163.1, 101.1)
- added R21: 150kΩ, PCM_JLCPCB:R_0805, F.Cu at (154.6, 106.7)
- added R22: 100kΩ, PCM_JLCPCB:R_0805, F.Cu at (182.0, 95.0)
- added R23: 3.3kΩ, PCM_JLCPCB:R_0805, F.Cu at (99.3, 48.3)
- added R24: 3.3kΩ, PCM_JLCPCB:R_0805, F.Cu at (99.3, 51.2)
- added R25: 4.7kΩ, PCM_JLCPCB:R_0805, F.Cu at (121.8, 47.0)
- added R26: 4.7kΩ, PCM_JLCPCB:R_0805, F.Cu at (121.8, 50.0)
- added R27: 0Ω, PCM_JLCPCB:R_0805, F.Cu at (168.8, 117.5)
- added R28: 0Ω, PCM_JLCPCB:R_0805, F.Cu at (170.8, 117.5)
- added R3: 1Ω 1W, Resistor_SMD:R_2512_6332Metric_Pad1.40x3.35mm_HandSolder, F.Cu at (160.8, 104.1)
- added R4: 100kΩ, PCM_JLCPCB:R_0805, F.Cu at (154.6, 104.7)
- added R5: 2.2kΩ, PCM_JLCPCB:R_0805, F.Cu at (99.3, 33.5)
- added R6: 10Ω, PCM_JLCPCB:R_0805, F.Cu at (194.1, 96.3)
- added R7: 1.5kΩ, PCM_JLCPCB:R_0805, F.Cu at (149.9, 98.2)
- added R8: 750Ω, PCM_JLCPCB:R_0805, F.Cu at (151.9, 98.2)
- added R9: 100Ω, PCM_JLCPCB:R_0805, F.Cu at (180.0, 91.6)
- added SW2: Trigger, Connector_PinHeader_2.54mm:PinHeader_1x02_P2.54mm_Vertical, F.Cu at (117.1, 44.0)
- added SW3: Reload, Connector_PinHeader_2.54mm:PinHeader_1x02_P2.54mm_Vertical, F.Cu at (117.0, 50.2)
- added SW4: SW_Push, Button_Switch_SMD:SW_SPST_CK_RS282G05A3, B.Cu at (199.0, 120.1)
- added SW5: SW_Push_DPDT, nnaf:MHPS2266, B.Cu at (202.1, 97.6)
- added SW6: SW_Push, Button_Switch_SMD:SW_SPST_CK_RS282G05A3, B.Cu at (169.0, 107.0)
- added TP1: TestPoint, TestPoint:TestPoint_Pad_D3.0mm, F.Cu at (206.2, 75.5)
- added TP2: TestPoint, TestPoint:TestPoint_Pad_D3.0mm, F.Cu at (184.3, 91.1)
- added U1: AMS1117, PCM_JLCPCB:SOT-223-3_L6.5-W3.4-P2.30-LS7.0-BR, F.Cu at (189.9, 100.0)
- added U2: ESP32-S3-WROOM-1, RF_Module:ESP32-S3-WROOM-1, F.Cu at (183.6, 118.7)
- added U3: TPS54302, Package_TO_SOT_SMD:SOT-23-6, F.Cu at (176.1, 95.0)
- added U4: MAX98357A, Package_DFN_QFN:TQFN-16-1EP_3x3mm_P0.5mm_EP1.23x1.23mm, B.Cu at (168.7, 113.0)
- added U5: MCP4531T-103E_MS, MCP4561_103E_MS:SOP65P490X110-8N, B.Cu at (150.3, 103.5)
- added U6: LIS3DH, Package_LGA:LGA-16_3x3mm_P0.5mm_LayoutBorder3x5y, F.Cu at (171.7, 98.6)
- added U7: LMV321IDBVR, PCM_JLCPCB:SOT-23-5_L3.0-W1.7-P0.95-LS2.8-BR, F.Cu at (178.1, 100.1)
- added U8: LMV321IDBVR, PCM_JLCPCB:SOT-23-5_L3.0-W1.7-P0.95-LS2.8-BR, F.Cu at (154.6, 101.8)
- added U9: OPA197IDR, opa197idr:D0008A-IPC_A, F.Cu at (156.9, 97.5)
Routing:
- net GND: track 0.00 -> 127.5 mm, vias 0 -> 20
- net Net-(BT2-+): track 0.00 -> 71.8 mm
- net SDA: track 0.00 -> 66.8 mm, vias 0 -> 2
- net +BATT: track 0.00 -> 54.0 mm, vias 0 -> 1
- net SCL: track 0.00 -> 51.6 mm, vias 0 -> 2
- net +3.3V: track 0.00 -> 50.1 mm, vias 0 -> 9
- net Net-(C12-Pad1): track 0.00 -> 36.8 mm, vias 0 -> 1
- net IO21: track 0.00 -> 35.1 mm, vias 0 -> 1
- net LIS3DH_Int1: track 0.00 -> 22.7 mm
- net /µC/EN: track 0.00 -> 20.2 mm, vias 0 -> 1
- net Net-(U8-+): track 0.00 -> 20.2 mm, vias 0 -> 1
- net Net-(Q2-D): track 0.00 -> 18.8 mm
- net Net-(J2-Pin_1): track 0.00 -> 15.9 mm
- net +5V: track 0.00 -> 15.5 mm
- net LIS3DH_Int2: track 0.00 -> 15.3 mm
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- added copper zone on In2.Cu, net +3.3V
- added copper zone on In1.Cu, net GND
Other:
- board outline added: 56 x 38 mm
- copper layers 2 -> 4

Commit message: pcb didn't commit correctly
Parts:
- removed C21: 220µF, Capacitor_THT:CP_Radial_D6.3mm_P2.50mm
- removed C23: 100nF, PCM_JLCPCB:C_1206
- removed C25: 22uF, PCM_JLCPCB:C_1206
- removed Camera_Interface1: Conn_02x08_Counter_Clockwise, Connector_JST:JST_PH_B16B-PH-SM4-TB_1x16-1MP_P2.00mm_Vertical
- removed JP5: Jumper, Jumper:SolderJumper-3_P1.3mm_Bridged12_RoundedPad1.0x1.5mm_NumberLabels
- added PN1: ~, PCM_JLCPCB:Part_Num_JLCPCB, B.Cu at (183.8, 122.3)
- added REF**: ToolingHole_1.152mm, MountingHole:ToolingHole_1.152mm, F.Cu at (199.0, 103.3)
- added REF**: ToolingHole_1.152mm, MountingHole:ToolingHole_1.152mm, F.Cu at (199.5, 123.5)
- added REF**: ToolingHole_1.152mm, MountingHole:ToolingHole_1.152mm, F.Cu at (175.0, 90.5)
- added REF**: ToolingHole_1.152mm, MountingHole:ToolingHole_1.152mm, F.Cu at (146.5, 115.5)
- added REF**: ToolingHole_1.152mm, MountingHole:ToolingHole_1.152mm, F.Cu at (147.5, 89.5)
- added TP3: IO22, TestPoint:TestPoint_Pad_D1.5mm, F.Cu at (149.3, 104.8)
- added TP4: Ir-current, TestPoint:TestPoint_Pad_D1.5mm, F.Cu at (151.6, 94.7)
- added TP5: Gnd, TestPoint:TestPoint_Pad_D2.0mm, F.Cu at (199.1, 96.0)
- added TP6: ir-signal, TestPoint:TestPoint_Pad_D1.5mm, F.Cu at (157.2, 114.8)
- added TP7: TestPoint, TestPoint:TestPoint_Pad_D1.5mm, F.Cu at (199.7, 100.7)
- C20, J8, JP6, JP7: moved to B.Cu
- J3: footprint Connector_JST:JST_PH_S6B-PH-SM4-TB_1x06-1MP_P2.00mm_Horizontal -> Connector_JST:JST_PH_B6B-PH-SM4-TB_1x06-1MP_P2.00mm_Vertical
- J5, J6: footprint Connector_JST:JST_PH_S2B-PH-SM4-TB_1x02-1MP_P2.00mm_Horizontal -> Connector_JST:JST_PH_B2B-PH-SM4-TB_1x02-1MP_P2.00mm_Vertical; moved to B.Cu
- J7: footprint Connector_JST:JST_PH_S2B-PH-SM4-TB_1x02-1MP_P2.00mm_Horizontal -> Connector_JST:JST_PH_B2B-PH-SM4-TB_1x02-1MP_P2.00mm_Vertical
- L1: footprint Inductor_SMD:L_Coilcraft_LPS5030 -> Inductor_SMD:L_Coilcraft_LPS4018
- TP1: value TestPoint -> 3.3V; footprint TestPoint:TestPoint_Pad_D3.0mm -> TestPoint:TestPoint_Pad_D2.0mm
- TP2: value TestPoint -> total-current; footprint TestPoint:TestPoint_Pad_D3.0mm -> TestPoint:TestPoint_Pad_D1.5mm
- U4: moved to F.Cu
- moved D1 105.4 mm to (171.8, 122.6), turned to -90 degrees
- moved JP6 104.0 mm to (189.8, 101.5)
- moved JP7 103.3 mm to (189.8, 104.0)
- moved R1 101.9 mm to (198.5, 108.4), turned to 180 degrees
- moved R11 101.8 mm to (198.5, 111.1), turned to 180 degrees
- moved R23 99.8 mm to (168.4, 120.3), turned to 180 degrees
- moved J8 99.6 mm to (182.2, 97.6)
- moved Q8 98.2 mm to (168.7, 123.1)
- moved R5 97.6 mm to (158.3, 111.3)
- moved R24 89.7 mm to (163.6, 113.8)
- moved D2 87.7 mm to (163.1, 110.5), turned to 90 degrees
- moved Q9 83.6 mm to (166.3, 111.1), turned to 180 degrees
- moved JP1 81.5 mm to (152.7, 112.9), turned to 90 degrees
- moved C32 80.6 mm to (152.4, 109.5), turned to 90 degrees
- moved C18 79.4 mm to (155.2, 93.4), turned to 180 degrees
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Connections:
- JP7 pad 3: IO43 -> IO11
- R24 pad 1: IO44D -> IO44
- U2 pad 10: CAM_D6 -> unconnected-(U2-IO17-Pad10)
- U2 pad 11: CAM_D7 -> unconnected-(U2-IO18-Pad11)
- U2 pad 15: LIS3DH_Int1 -> unconnected-(U2-IO3-Pad15)
- U2 pad 17: CAM_HS -> unconnected-(U2-IO9-Pad17)
- U2 pad 18: CAM_PC -> unconnected-(U2-IO10-Pad18)
- U2 pad 19: CAM_PD -> IO11
- U2 pad 20: CAM_VS -> LIS3DH_Int1
- U2 pad 24: IR_Signal -> unconnected-(U2-IO47-Pad24)
- U2 pad 25: Hit_Lamp -> unconnected-(U2-IO48-Pad25)
- U2 pad 36: /µC/IO44 -> IO44
- U2 pad 4: CAM_D0 -> unconnected-(U2-IO4-Pad4)
- U2 pad 5: CAM_D1 -> Hit_Lamp
- U2 pad 6: CAM_D2 -> IR_Signal
- U2 pad 7: CAM_D3 -> unconnected-(U2-IO7-Pad7)
- U2 pad 8: CAM_D4 -> unconnected-(U2-IO15-Pad8)
- U2 pad 9: CAM_D5 -> unconnected-(U2-IO16-Pad9)
Routing:
- net +BATT: track 54.0 -> 142.9 mm, vias 1 -> 5
- net IR_Signal: track 0.00 -> 74.2 mm, vias 0 -> 2
- net IR_ADC: track 4.32 -> 50.2 mm, vias 0 -> 2
- net Hit_Lamp: track 0.00 -> 45.1 mm, vias 0 -> 2
- net +3.3V: track 50.1 -> 92.7 mm, vias 9 -> 12
- net IO36: track 0.00 -> 40.3 mm, vias 0 -> 1
- net IO35: track 0.00 -> 37.7 mm, vias 0 -> 1
- net GND: track 127.5 -> 164.0 mm, vias 20 -> 29
- net Batt_ADC: track 2.60 -> 36.7 mm, vias 0 -> 4
- net Reload: track 0.00 -> 31.2 mm, vias 0 -> 1
- net Trigger: track 0.00 -> 28.0 mm, vias 0 -> 1
- net Net-(J6-Pin_1): track 0.00 -> 25.1 mm, vias 0 -> 1
- net SCL: track 51.6 -> 75.4 mm, vias 2 -> 4
- net SDA: track 66.8 -> 89.5 mm, vias 2 -> 3
- net IO44: track 0.00 -> 20.8 mm
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Other:
- outline, holes or cut-outs redrawn
- board text added: "3.3V"
- board text added: "Batt_ADC"
- board text added: "GND"
- board text added: "ir-shoot"
- board text added: "ir-signal"
- board text added: "ir_current"
- board text added: "total_current"
