File: in_out_puts.kicad_sch (KiCad schematic)
At the start: 45 parts, among them J2 Conn_01x02_Socket, J3 Dome, J5 Motor1, J6 Motor2, J7 Speaker, J8 Conn_01x07, J9 IR-LED, Q1 IRLML6344TRPBF, Q8 S9014, Q9 S9014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

Commit message: pcb didn't commit correctly
Parts:
- removed Camera_Interface1: Conn_02x08_Counter_Clockwise, Connector_JST:JST_PH_B16B-PH-SM4-TB_1x16-1MP_P2.00mm_Vertical, symbol Connector_Generic:Conn_02x08_Counter_Clockwise
- added TP3: IO22, TestPoint:TestPoint_Pad_D1.5mm, symbol Connector:TestPoint
- added TP4: Ir-current, TestPoint:TestPoint_Pad_D1.5mm, symbol Connector:TestPoint
- added TP5: Gnd, TestPoint:TestPoint_Pad_D2.0mm, symbol Connector:TestPoint
- added TP6: ir-signal, TestPoint:TestPoint_Pad_D1.5mm, symbol Connector:TestPoint
- J3: footprint Connector_JST:JST_PH_S6B-PH-SM4-TB_1x06-1MP_P2.00mm_Horizontal -> Connector_JST:JST_PH_B6B-PH-SM4-TB_1x06-1MP_P2.00mm_Vertical
- J5, J6, J7: footprint Connector_JST:JST_PH_S2B-PH-SM4-TB_1x02-1MP_P2.00mm_Horizontal -> Connector_JST:JST_PH_B2B-PH-SM4-TB_1x02-1MP_P2.00mm_Vertical
Connections:
- net GND: now also TP5.1
- net IO21: now also TP3.1
- net IO43: no longer JP7.3 (B)
- net IR_Signal: now also TP6.1
- net at C27.2, Q1.2, R3.1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: now also TP4.1
- net IO44D renamed IO44
- new net IO11: JP7.3 (B)
Other:
- note removed: "CAM_Interface"
- note removed: "Interface for Adafruit OV5640 Camera Breakouts"
- moved on the sheet: C32, C33
