File: in_out_puts.kicad_sch (KiCad schematic)
At the start: 48 parts, among them J2 Conn_01x02_Socket, J3 Dome, J5 Motor1, J6 Motor2, J7 Speaker, J8 Conn_01x07, J9 IR-LED, Q1 IRLML6344TRPBF, Q8 S9014, Q9 S9014, SW2 Trigger, SW3 Reload, U4 MAX98357A, U5 MCP4531T-103E_MS, U6 LIS3DH, U8 LMV321IDBVR, U9 OPA197IDR

Commit message: .
Parts:
- U5: value MCP4531T-103E_MS -> MCP4561T-103E_MS
Changed lines of the file:
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@@
 			)
 		)
-		(property "Datasheet" ""
+		(property "Datasheet" "https://www.mouser.at/datasheet/3/70/1/Infineon_IRLML6344_DataSheet_v01_01_EN.pdf"
 			(at 76.2 161.29 0)
 			(effects
@@
 			)
 		)
-		(property "Value" "MCP4531T-103E_MS"
+		(property "Value" "MCP4561T-103E_MS"
 			(at 40.132 148.336 0)
 			(effects
