File: µC.kicad_sch (KiCad schematic)
At the start: 17 parts, among them J4 USB_C_Receptacle_USB2.0_14P, SW4 SW_Push, SW6 SW_Push, U2 ESP32-S3-WROOM-1

Commit message: .
Parts:
- added R13: 10kΩ, PCM_JLCPCB:R_0805, symbol PCM_JLCPCB-Resistors:0805,10kΩ
Connections:
- net GND: now also R13.2
- net at U2.16 (IO46): now also R13.1
- no-connect marks 14 -> 13
